Commit message: fix: 使用扁平dist目录结构，HACS可以下载所有文件

File: dist/reachy-mini.urdf (robot description, URDF)
Before this commit: robot robot, 45 links, 44 joints
Links:
- link body_down_3dprint: geometry collision mesh filename=5w_speaker.stl; collision mesh filename=b3b_eh.stl
- link body_foot_3dprint: geometry collision mesh filename=body_foot_3dprint.stl; collision mesh filename=body_turning_3dprint.stl
- link dc15_a01_horn_dummy: geometry collision mesh filename=dc15_a01_horn_dummy.stl; collision mesh filename=mp01062_stewart_arm_3.stl
- link dc15_a01_horn_dummy_2: geometry collision mesh filename=dc15_a01_horn_dummy.stl; collision mesh filename=mp01062_stewart_arm_3.stl
- link dc15_a01_horn_dummy_3: geometry collision mesh filename=dc15_a01_horn_dummy.stl; collision mesh filename=mp01062_stewart_arm_3.stl
- link dc15_a01_horn_dummy_4: geometry collision mesh filename=dc15_a01_horn_dummy.stl; collision mesh filename=mp01062_stewart_arm_3.stl
- link dc15_a01_horn_dummy_5: geometry collision mesh filename=dc15_a01_horn_dummy.stl; collision mesh filename=mp01062_stewart_arm_3.stl
- link dc15_a01_horn_dummy_6: geometry collision mesh filename=dc15_a01_horn_dummy.stl; collision mesh filename=mp01062_stewart_arm_3.stl
- link dc15_a01_horn_dummy_7: geometry collision mesh filename=antenna.stl; collision mesh filename=antenna_body_3dprint.stl
- link dc15_a01_horn_dummy_8: geometry collision mesh filename=antenna.stl; collision mesh filename=antenna_body_3dprint.stl
- link stewart_link_rod: geometry collision mesh filename=stewart_link_rod.stl; visual mesh filename=stewart_link_rod.stl
- link stewart_link_rod_2: geometry collision mesh filename=stewart_link_rod.stl; visual mesh filename=stewart_link_rod.stl
- link stewart_link_rod_3: geometry collision mesh filename=stewart_link_rod.stl; visual mesh filename=stewart_link_rod.stl
- link stewart_link_rod_4: geometry collision mesh filename=stewart_link_rod.stl; visual mesh filename=stewart_link_rod.stl
- link stewart_link_rod_5: geometry collision mesh filename=stewart_link_rod.stl; visual mesh filename=stewart_link_rod.stl
- link stewart_link_rod_6: geometry collision mesh filename=stewart_link_rod.stl; visual mesh filename=stewart_link_rod.stl
- link xl_330: geometry collision mesh filename=antenna_holder_l_3dprint.stl; collision mesh filename=antenna_holder_r_3dprint.stl
